File: Boost.brd (EAGLE design)
At the start: 100 x 80 mm, 44 parts, among them IC1 4069N, Q1 2N3904, Q2 2N3906, Q3 2N3904, Q4 2N3906, Q5 2N3904, Q6 2N3904, Q7 P3N100XI

Commit message: board work
Parts:
- removed L1: (no value), rcl:0204/5
- added C14, C15, C16, C17, C18, C19, C20, C21, C22, C23, C24, C25: (no value), rcl:C050-024X044
- added D10, D11, D12, D13, D14, D15: 1N4004, diode:DO41-10
- added IC2: (no value), v-reg:78XXS
- IC1: value 4069N -> 74LS14N; device 40xx:DIL14 -> 74xx-us:DIL14
- Q7: value P3N100XI -> TIP120; device transistor-power:IW221 -> transistor-power:TO220AH
- moved C13 297.1 mm to (142.2, 49.5), turned to 270 degrees
- moved D7 241.1 mm to (166.4, 43.2), turned to 270 degrees
- moved C11 238.8 mm to (-8.89, 54.6), turned to 180 degrees
- moved Q7 234.4 mm to (156.2, 41.9)
- moved R10 233.7 mm to (143.5, 35.6)
- moved C9 232.3 mm to (148.6, 49.5), turned to 270 degrees
- moved C7 231.9 mm to (160.0, 49.5), turned to 270 degrees
- moved C8 231.6 mm to (153.7, 49.5), turned to 270 degrees
- moved R12 229.9 mm to (-10.2, 50.8)
- moved C12 224.9 mm to (-1.27, 22.9), turned to 90 degrees
- moved D8 218.5 mm to (-10.2, 47.0)
- moved R13 216.0 mm to (-11.4, 19.1)
- moved C10 215.2 mm to (-22.9, 48.3)
- moved D9 214.7 mm to (-11.4, 25.4)
- moved R11 207.8 mm to (-22.9, 45.7), turned to 180 degrees
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Connections:
- removed net N$10: C2.2, C4.2, Q3.1, Q4.1
- removed net N$28: C13.1, C7.1, C8.1, C9.1, D7.C, L1.1, R7.2
- removed net N$7: D7.A, L1.2, Q7.D
- removed net VDD: IC1.14
- removed net VSS: IC1.7
- new net +5V: C25.1, IC1.14, IC2.OUT
- new net N$30: C15.2, C16.2, C2.2, C20.2, C22.2, C4.2, Q3.1, Q4.1
- new net SOL-HIGH: C13.1, C7.1, C8.1, C9.1, D7.C, R7.2
- new net SOL-LOW: D7.A, Q7.C
- net +12V: now also C24.1, D10.A, IC2.IN
- net +5V1: now also C15.1, C22.1, D11.C, D12.A
- net GND: now also C24.2, C25.2, IC1.7, IC2.GND, Q7.E; no longer Q7.S
- net N$11: now also C17.1, C19.1, D14.A, D15.C
- net N$12: now also D14.C
- net N$13: now also C14.2, C17.2, C18.2, C19.2, C21.2, C23.2
- net N$18: now also IC1.6; no longer IC1.12
- net N$19: now also Q7.B; no longer Q7.G
- net N$2: now also C14.1, C23.1, D10.C, D11.A
- net N$21: now also IC1.1, IC1.11, IC1.12; no longer IC1.2, IC1.3, IC1.5
- net N$22: now also IC1.13; no longer IC1.1
- net N$24: now also IC1.10; no longer IC1.6
- net N$25: now also IC1.5; no longer IC1.13
- net N$26: now also IC1.4; no longer IC1.10
- net N$27: now also IC1.2, IC1.3; no longer IC1.11, IC1.4
- net N$8: now also C18.1, C21.1, D12.C, D13.A
- net N$9: now also C16.1, C20.1, D13.C, D15.A
Routing:
- net +12V: track 36.2 -> 153.8 mm
- net N$30: track 0.00 -> 106.0 mm
- net N$13: track 21.4 -> 109.5 mm, vias 0 -> 1
- net N$1: track 2.54 -> 59.6 mm
- net SOL-HIGH: track 0.00 -> 47.8 mm
- net GND: track 20.4 -> 52.9 mm, vias 1 -> 0
- net N$25: track 0.00 -> 31.6 mm
- net N$11: track 0.00 -> 31.3 mm
- net N$8: track 0.00 -> 31.3 mm
- net N$9: track 0.00 -> 30.7 mm
- net N$3: track 2.54 -> 28.8 mm, vias 1 -> 0
- net +5V: track 0.00 -> 23.3 mm
- net N$16: track 0.00 -> 21.9 mm
- net N$12: track 0.00 -> 20.3 mm
- net N$23: track 0.00 -> 20.2 mm
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- added copper zone on layer 16, net GND
Other:
- board size 100 x 80 mm -> 276.5 x 80 mm

Commit message: board design
Parts:
- removed Q7: TIP120, transistor-power:TO220AH
- added Q8: IRF530, transistor-power:TO220BV
- moved D7 109.4 mm to (61.0, 14.0), turned to 90 degrees
- moved C7 102.9 mm to (66.0, 7.62), turned to 90 degrees
- moved C8 92.6 mm to (71.1, 7.62), turned to 90 degrees
- moved C9 83.6 mm to (76.2, 7.62), turned to 90 degrees
- moved R10 76.2 mm to (67.3, 35.6), turned to 180 degrees
- moved C13 74.0 mm to (81.3, 7.62), turned to 90 degrees
- moved C24 72.6 mm to (17.8, 11.4), turned to 180 degrees
- moved R7 70.1 mm to (86.4, 7.62), turned to 270 degrees
- moved C6 67.3 mm to (71.1, 16.5), turned to 90 degrees
- moved IC2 65.6 mm to (14.0, 2.54), turned to 180 degrees
- moved C25 62.1 mm to (10.2, 11.4), turned to 0 degrees
- moved D14 59.5 mm to (80.0, 15.2), turned to 0 degrees
- moved D6 51.4 mm to (80.0, 20.3), turned to 0 degrees
- moved D15 50.1 mm to (92.7, 15.2), turned to 0 degrees
- moved C19 45.4 mm to (73.7, 29.2), turned to 90 degrees
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Connections:
- net GND: now also Q8.S; no longer Q7.E
- net N$19: now also Q8.G; no longer Q7.B
- net SOL-LOW: now also Q8.D; no longer Q7.C
Routing:
- net GND: track 52.9 -> 11.7 mm
- net N$9: track 30.7 -> 66.9 mm
- net +12V: track 153.8 -> 123.2 mm
- net +5V: track 23.3 -> 38.5 mm
- net N$30: track 106.0 -> 120.0 mm
- net N$13: track 109.5 -> 95.6 mm
- net SOL-HIGH: track 47.8 -> 35.1 mm, vias 0 -> 1
- net N$16: track 21.9 -> 10.5 mm
- net N$21: track 18.4 -> 29.5 mm
- net N$19: track 5.08 -> 13.5 mm
- net N$17: track 4.07 -> 9.68 mm
- net SOL-LOW: track 14.8 -> 20.4 mm, vias 0 -> 1
- net N$24: track 13.5 -> 18.6 mm
- net N$18: track 18.1 -> 13.8 mm
- net N$22: track 13.0 -> 17.3 mm
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Other:
- board size 276.5 x 80 mm -> 100 x 67.3 mm
