File: Boost.sch (EAGLE design)
At the start: 62 parts, among them IC1 74LS14N, Q1 2N3904, Q2 2N3906, Q3 2N3904, Q4 2N3906, Q5 2N3904, Q6 2N3904, Q7 TIP120

Commit message: board design
Parts:
- removed Q7: TIP120, transistor-power:TIP120
- added Q8: IRF530, transistor-power:IRF530
Connections:
- net GND: now also Q8.S; no longer Q7.E
- net N$19: now also Q8.G; no longer Q7.B
- net SOL-LOW: now also Q8.D; no longer Q7.C
Changed lines of the file:
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@@
 <part name="GND12" library="supply1" library_urn="urn:adsk.eagle:library:371" deviceset="GND" device=""/>
 <part name="GND13" library="supply1" library_urn="urn:adsk.eagle:library:371" deviceset="GND" device=""/>
-<part name="Q7" library="transistor-power" library_urn="urn:adsk.eagle:library:400" deviceset="TIP120" device="" package3d_urn="urn:adsk.eagle:package:29488/1"/>
+<part name="Q8" library="transistor-power" library_urn="urn:adsk.eagle:library:400" deviceset="IRF530" device="" package3d_urn="urn:adsk.eagle:package:29484/3"/>
 </parts>
 <sheets>
@@
 <attribute name="VALUE" x="-170.18" y="43.18" size="1.778" layer="96"/>
 </instance>
-<instance part="Q7" gate="1" x="226.06" y="-5.08" smashed="yes">
-<attribute name="NAME" x="231.14" y="-2.54" size="1.778" layer="95"/>
-<attribute name="VALUE" x="231.14" y="-5.08" size="1.778" layer="96"/>
+<instance part="Q8" gate="G$1" x="226.06" y="-5.08" smashed="yes">
+<attribute name="NAME" x="233.68" y="-2.54" size="1.778" layer="95"/>
+<attribute name="VALUE" x="233.68" y="-5.08" size="1.778" layer="96"/>
 </instance>
 </instances>
@@
 <pinref part="GND6" gate="1" pin="GND"/>
 <wire x1="228.6" y1="-15.24" x2="228.6" y2="-10.16" width="0.1524" layer="91"/>
-<pinref part="Q7" gate="1" pin="E"/>
+<pinref part="Q8" gate="G$1" pin="S"/>
 </segment>
 <segment>
@@
 <junction x="228.6" y="5.08"/>
 <label x="228.6" y="7.62" size="1.27" layer="95" rot="R90" xref="yes"/>
-<pinref part="Q7" gate="1" pin="C"/>
+<pinref part="Q8" gate="G$1" pin="D"/>
 </segment>
 </net>
 <net name="N$19" class="0">
 <segment>
-<wire x1="223.52" y1="-5.08" x2="213.36" y2="-5.08" width="0.1524" layer="91"/>
 <pinref part="R10" gate="G$1" pin="2"/>
-<pinref part="Q7" gate="1" pin="B"/>
-</segment>
-</net>
+<pinref part="Q8" gate="G$1" pin="G"/>
+<wire x1="215.9" y1="-5.08" x2="213.36" y2="-5.08" width="0.1524" layer="91"/>
+<wire x1="223.52" y1="-7.62" x2="215.9" y2="-7.62" width="0.1524" layer="91"/>
+<wire x1="215.9" y1="-7.62" x2="215.9" y2="-5.08" width="0.1524" layer="91"/>
+</segment>
+</net>
